Commit message: correct ucollada_urdf

File: urdf/ur5.urdf (robot description, URDF)
Before this commit: robot ur5, 11 links, 10 joints
Joints:
- removed joint wrist_3_link-tool0_fixed_joint
- added joint wrist_3_passive_joint: type fixed, parent wrist_3_link, child tool0, origin xyz=0 0 0 rpy=0 0 0
- joint ee_fixed_joint: origin xyz=0.0 0.0823 0.0 rpy=0.0 0.0 1.57079632679 -> xyz=0.0 0.0 0.0 rpy=0.0 -1.57079632679 1.57079632679
- joint elbow_joint: axis 0 1 0 -> 0 0 1; origin xyz=0.0 -0.1197 0.425 rpy=0.0 0.0 0.0 -> xyz=-0.425389617445 0 0 rpy=3.14037678529 3.1396825367 -3.14150448323
- joint shoulder_lift_joint: axis 0 1 0 -> 0 0 1; limit lower=-6.28318530718 upper=6.28318530718 effort=150.0 velocity=3.15 -> lower=-3.14159265359 upper=3.14159265359 effort=150.0 velocity=3.15; origin xyz=0.0 0.13585 0.0 rpy=0.0 1.57079632679 0.0 -> xyz=6.33636237145e-05 0 0 rpy=1.57034854095 0 2.71904566699e-05
- joint shoulder_pan_joint: limit lower=-6.28318530718 upper=6.28318530718 effort=150.0 velocity=3.15 -> lower=-3.14159265359 upper=3.14159265359 effort=150.0 velocity=3.15; origin xyz=0.0 0.0 0.089159 rpy=0.0 0.0 0.0 -> xyz=0 0 0.0893895156178 rpy=0 0 3.14160348585
- joint wrist_1_joint: axis 0 1 0 -> 0 0 1; limit lower=-6.28318530718 upper=6.28318530718 effort=28.0 velocity=3.2 -> lower=-3.14159265359 upper=3.14159265359 effort=28.0 velocity=3.2; origin xyz=0.0 0.0 0.39225 rpy=0.0 1.57079632679 0.0 -> xyz=-0.392506907374 0.00031185980036 0.11018899121 rpy=3.13876243467 -3.14043849801 -3.14155879866
- joint wrist_2_joint: limit lower=-6.28318530718 upper=6.28318530718 effort=28.0 velocity=3.2 -> lower=-3.14159265359 upper=3.14159265359 effort=28.0 velocity=3.2; origin xyz=0.0 0.093 0.0 rpy=0.0 0.0 0.0 -> xyz=3.3323577063e-05 -0.0947783958619 4.33505448434e-06 rpy=1.57075058795 0 5.49664109762e-05
- joint wrist_3_joint: axis 0 1 0 -> 0 0 1; limit lower=-6.28318530718 upper=6.28318530718 effort=28.0 velocity=3.2 -> lower=-3.14159265359 upper=3.14159265359 effort=28.0 velocity=3.2; origin xyz=0.0 0.0 0.09465 rpy=0.0 0.0 0.0 -> xyz=5.02447530839e-05 0.0824869782666 -2.10041838233e-06 rpy=1.57077086316 3.14159265359 -3.14150915496

File: urdf/ur5.urdf.xacro (robot description, xacro)
@@ -4,4 +4,4 @@
   <xacro:arg name="kinematics_config" default="$(find ur5_ikfast_build)/my_robot_calibration.yaml"/>
   <!-- ur5 -->
-  <xacro:include filename="$(find ur_description)/urdf/ur5_robot.urdf.xacro" />
+  <xacro:include filename="$(find ur_description)/urdf/ur5_joint_limited_robot.urdf.xacro" />
 </robot>

Commit message: update .dae

File: urdf/ur5.urdf (robot description, URDF)
Before this commit: robot ur5, 11 links, 10 joints
Joints:
- joint shoulder_lift_joint: limit lower=-3.14159265359 upper=3.14159265359 effort=150.0 velocity=3.15 -> lower=-6.28318530718 upper=6.28318530718 effort=150.0 velocity=3.15
- joint shoulder_pan_joint: limit lower=-3.14159265359 upper=3.14159265359 effort=150.0 velocity=3.15 -> lower=-6.28318530718 upper=6.28318530718 effort=150.0 velocity=3.15
- joint wrist_1_joint: limit lower=-3.14159265359 upper=3.14159265359 effort=28.0 velocity=3.2 -> lower=-6.28318530718 upper=6.28318530718 effort=28.0 velocity=3.2
- joint wrist_2_joint: limit lower=-3.14159265359 upper=3.14159265359 effort=28.0 velocity=3.2 -> lower=-6.28318530718 upper=6.28318530718 effort=28.0 velocity=3.2
- joint wrist_3_joint: limit lower=-3.14159265359 upper=3.14159265359 effort=28.0 velocity=3.2 -> lower=-6.28318530718 upper=6.28318530718 effort=28.0 velocity=3.2

Commit message: without calibration

File: urdf/ur5.urdf (robot description, URDF)
Before this commit: robot ur5, 11 links, 10 joints
Joints:
- joint elbow_joint: origin xyz=-0.425389617445 0 0 rpy=3.14037678529 3.1396825367 -3.14150448323 -> xyz=-0.425 0 0 rpy=0 0 0
- joint shoulder_lift_joint: origin xyz=6.33636237145e-05 0 0 rpy=1.57034854095 0 2.71904566699e-05 -> xyz=0 0 0 rpy=1.570796327 0 0
- joint shoulder_pan_joint: origin xyz=0 0 0.0893895156178 rpy=0 0 3.14160348585 -> xyz=0 0 0.089159 rpy=0 0 3.14159265359
- joint wrist_1_joint: origin xyz=-0.392506907374 0.00031185980036 0.11018899121 rpy=3.13876243467 -3.14043849801 -3.14155879866 -> xyz=-0.39225 0 0.10915 rpy=0 0 0
- joint wrist_2_joint: origin xyz=3.3323577063e-05 -0.0947783958619 4.33505448434e-06 rpy=1.57075058795 0 5.49664109762e-05 -> xyz=0 -0.09465 -1.9413039509e-11 rpy=1.570796327 0 0
- joint wrist_3_joint: origin xyz=5.02447530839e-05 0.0824869782666 -2.10041838233e-06 rpy=1.57077086316 3.14159265359 -3.14150915496 -> xyz=0 0.0823 -1.68800121668e-11 rpy=1.57079632659 3.14159265359 3.14159265359

Commit message: ikfast success

File: urdf/ur5.urdf (robot description, URDF)
Before this commit: robot ur5, 11 links, 10 joints
Joints:
- removed joint wrist_3_passive_joint
- added joint wrist_3_link-tool0_fixed_joint: type fixed, parent wrist_3_link, child tool0, origin xyz=0 0.0823 0 rpy=-1.57079632679 0 0
- joint ee_fixed_joint: origin xyz=0.0 0.0 0.0 rpy=0.0 -1.57079632679 1.57079632679 -> xyz=0.0 0.0823 0.0 rpy=0.0 0.0 1.57079632679
- joint elbow_joint: axis 0 0 1 -> 0 1 0; origin xyz=-0.425 0 0 rpy=0 0 0 -> xyz=0.0 -0.1197 0.425 rpy=0.0 0.0 0.0
- joint shoulder_lift_joint: axis 0 0 1 -> 0 1 0; origin xyz=0 0 0 rpy=1.570796327 0 0 -> xyz=0.0 0.13585 0.0 rpy=0.0 1.57079632679 0.0
- joint shoulder_pan_joint: origin xyz=0 0 0.089159 rpy=0 0 3.14159265359 -> xyz=0.0 0.0 0.089159 rpy=0.0 0.0 0.0
- joint wrist_1_joint: axis 0 0 1 -> 0 1 0; origin xyz=-0.39225 0 0.10915 rpy=0 0 0 -> xyz=0.0 0.0 0.39225 rpy=0.0 1.57079632679 0.0
- joint wrist_2_joint: origin xyz=0 -0.09465 -1.9413039509e-11 rpy=1.570796327 0 0 -> xyz=0.0 0.093 0.0 rpy=0.0 0.0 0.0
- joint wrist_3_joint: axis 0 0 1 -> 0 1 0; origin xyz=0 0.0823 -1.68800121668e-11 rpy=1.57079632659 3.14159265359 3.14159265359 -> xyz=0.0 0.0 0.09465 rpy=0.0 0.0 0.0

Commit message: calibration xacro for openrave ikfast

File: urdf/ur5.urdf (robot description, URDF)
Before this commit: robot ur5, 11 links, 10 joints
Links:
- added link base_pre_link
- added link base_suf_link
- added link ee_pre_link
- added link forearm_pre_link
- added link forearm_suf_link
- added link shoulder_pre_link
- added link shoulder_suf_link
- added link upper_arm_pre_link
- added link upper_arm_suf_link
- added link wrist_1_pre_link
- added link wrist_1_suf_link
- added link wrist_2_pre_link
- added link wrist_2_suf_link
- added link wrist_3_pre_link
- added link wrist_3_suf_link
Joints:
- removed joint wrist_3_link-tool0_fixed_joint
- added joint base_pre_joint: type fixed, parent world, child base_pre_link, origin xyz=0.0 0.0 0.0 rpy=0.0 0.0 0.0
- added joint base_suf_joint: type fixed, parent base_link, child base_suf_link, origin xyz=0.0 0.0 0.0 rpy=0.0 0.0 -3.14159265359
- added joint ee_pre_joint: type fixed, parent wrist_3_suf_link, child ee_pre_link, origin xyz=0.0 0.0 0.0 rpy=0.0 -1.57079632679 1.57079632679
- added joint forearm_pre_joint: type fixed, parent upper_arm_suf_link, child forearm_pre_link, origin xyz=-0.425389617445 0 0 rpy=3.14037678529 3.1396825367 -3.14150448323
- added joint forearm_suf_joint: type fixed, parent forearm_link, child forearm_suf_link, origin xyz=0 -0.0165 0 rpy=-1.57079632679 1.57079632679 0
- added joint shoulder_pre_joint: type fixed, parent base_suf_link, child shoulder_pre_link, origin xyz=0 0 0.0893895156178 rpy=0 0 3.14160348585
- added joint shoulder_suf_joint: type fixed, parent shoulder_link, child shoulder_suf_link, origin xyz=0 0 0 rpy=0 0 -3.14159265359
- added joint upper_arm_pre_joint: type fixed, parent shoulder_suf_link, child upper_arm_pre_link, origin xyz=6.33636237145e-05 0 0 rpy=1.57034854095 0 2.71904566699e-05
- added joint upper_arm_suf_joint: type fixed, parent upper_arm_link, child upper_arm_suf_link, origin xyz=0 -0.136 0 rpy=-1.57079632679 1.57079632679 0
- added joint wrist_1_pre_joint: type fixed, parent forearm_suf_link, child wrist_1_pre_link, origin xyz=-0.392506907374 0.00031185980036 0.11018899121 rpy=3.13876243467 -3.14043849801 -3.14155879866
- added joint wrist_1_suf_joint: type fixed, parent wrist_1_link, child wrist_1_suf_link, origin xyz=0 0.093 0 rpy=-1.57079632679 0 0
- added joint wrist_2_pre_joint: type fixed, parent wrist_1_suf_link, child wrist_2_pre_link, origin xyz=3.3323577063e-05 -0.0947783958619 4.33505448434e-06 rpy=1.57075058795 0 5.49664109762e-05
- added joint wrist_2_suf_joint: type fixed, parent wrist_2_link, child wrist_2_suf_link, origin xyz=0 0 0.095 rpy=0 0 0
- added joint wrist_3_passive_joint: type fixed, parent wrist_3_link, child tool0, origin xyz=0 0 0 rpy=0 0 0
- added joint wrist_3_pre_joint: type fixed, parent wrist_2_suf_link, child wrist_3_pre_link, origin xyz=5.02447530839e-05 0.0824869782666 -2.10041838233e-06 rpy=1.57077086316 3.14159265359 -3.14150915496
- added joint wrist_3_suf_joint: type fixed, parent wrist_3_link, child wrist_3_suf_link, origin xyz=0 0.0818 0 rpy=-1.57079632679 0 0
- joint ee_fixed_joint: origin xyz=0.0 0.0823 0.0 rpy=0.0 0.0 1.57079632679 -> xyz=-0.01 0 0 rpy=0 0 0; parent wrist_3_link -> ee_pre_link
- joint elbow_joint: origin xyz=0.0 -0.1197 0.425 rpy=0.0 0.0 0.0 -> xyz=0 0 0.0165 rpy=1.57079632679 0 -1.57079632679; parent upper_arm_link -> forearm_pre_link
- joint shoulder_lift_joint: origin xyz=0.0 0.13585 0.0 rpy=0.0 1.57079632679 0.0 -> xyz=0 0 0.136 rpy=1.57079632679 0 -1.57079632679; parent shoulder_link -> upper_arm_pre_link
- joint shoulder_pan_joint: origin xyz=0.0 0.0 0.089159 rpy=0.0 0.0 0.0 -> xyz=0 0 0 rpy=0 0 3.14159265359; parent base_link -> shoulder_pre_link
- joint world_joint: origin xyz=0.0 0.0 0.0 rpy=0.0 0.0 0.0 -> xyz=0.0 0.0 0.0 rpy=0.0 0.0 3.14159265359; parent world -> base_pre_link
- joint wrist_1_joint: origin xyz=0.0 0.0 0.39225 rpy=0.0 1.57079632679 0.0 -> xyz=0 0 -0.093 rpy=1.57079632679 0 0; parent forearm_link -> wrist_1_pre_link
- joint wrist_2_joint: origin xyz=0.0 0.093 0.0 rpy=0.0 0.0 0.0 -> xyz=0 0 -0.095 rpy=0 0 0; parent wrist_1_link -> wrist_2_pre_link
- joint wrist_3_joint: origin xyz=0.0 0.0 0.09465 rpy=0.0 0.0 0.0 -> xyz=0 0 -0.0818 rpy=1.57079632679 0 0; parent wrist_2_link -> wrist_3_pre_link
