Commit message: CLOSE

File: bac/ur5.urdf.xacro (robot description, xacro)
@@ -43,5 +43,5 @@
     <xacro:property name="upper_arm_inertia_offset" value="0.136" />  <!-- measured from model -->
     <!-- This is for compatibility reasons, as transformation between base and base_link was always 180 degree in the ur_description -->
-    <xacro:property name="base_correction" value="${pi}" />
+    <xacro:property name="base_correction" value="${0}" />
     <link name="${prefix}base_link" >
       <visual>
@@ -309,5 +309,4 @@
       </visual>
       <collision>
-        <origin xyz="0 0 -0.095" rpy="0 0 0"/>
         <geometry>
           <mesh filename="package://ur_description/meshes/ur5/collision/wrist2.stl" />

File: bac/ur5_robot.urdf.xacro (robot description, xacro)
@@ -25,5 +25,5 @@
     <parent link="base_pre_link" />
     <child link = "base_link" />
-    <origin xyz="0.0 0.0 0.0" rpy="0.0 0.0 ${pi}" />
+    <origin xyz="0.0 0.0 0.0" rpy="0.0 0.0 ${0}" />
   </joint>
 </robot>

File: urdf/ur5.urdf (robot description, URDF)
Before this commit: robot ur5, 26 links, 25 joints
Joints:
- joint base_link-base_fixed_joint: origin xyz=0 0 0 rpy=0 0 -3.14159265359 -> xyz=0 0 0 rpy=0 0 0
- joint forearm_pre_joint: origin xyz=-0.425389617445 0 0 rpy=3.14037678529 3.1396825367 -3.14150448323 -> xyz=-0.425 0 0 rpy=0 0 0
- joint shoulder_pre_joint: origin xyz=0 0 0.0893895156178 rpy=0 0 3.14160348585 -> xyz=0 0 0.089159 rpy=0 0 0
- joint upper_arm_pre_joint: origin xyz=6.33636237145e-05 0 0 rpy=1.57034854095 0 2.71904566699e-05 -> xyz=0 0 0 rpy=1.570796327 0 0
- joint world_joint: origin xyz=0.0 0.0 0.0 rpy=0.0 0.0 3.14159265359 -> xyz=0.0 0.0 0.0 rpy=0.0 0.0 0
- joint wrist_1_pre_joint: origin xyz=-0.392506907374 0.00031185980036 0.11018899121 rpy=3.13876243467 -3.14043849801 -3.14155879866 -> xyz=-0.39225 0 0.10915 rpy=0 0 0
- joint wrist_2_pre_joint: origin xyz=3.3323577063e-05 -0.0947783958619 4.33505448434e-06 rpy=1.57075058795 0 5.49664109762e-05 -> xyz=0 -0.09465 -1.9413039509e-11 rpy=1.570796327 0 0
- joint wrist_3_pre_joint: origin xyz=5.02447530839e-05 0.0824869782666 -2.10041838233e-06 rpy=1.57077086316 3.14159265359 -3.14150915496 -> xyz=0 0.0823 -1.68800121668e-11 rpy=1.57079632659 3.14159265359 3.14159265359
